File: BigLatchingRelay/Electron/V1/PCB/BigLatchingRelay.brd (EAGLE design)
At the start: 99.1 x 31.2 mm, 13 parts, among them IC2 BD6211F

Commit message: Updated part identifiers and added BOMs
Parts:
- R1: value (none) -> 1k5
- renumbered IC2 to U3, U$2 to U2
